Commit message: Added separate sim w excavator only and added new excavator files

File: newton/auto_grading/assets/excavator.urdf (robot description, URDF)
Before this commit: robot MathScavator9000_flat.SLDASM, 5 links, 4 joints
Links:
- removed link base_chassis_link
- removed link boom_stick_link
- removed link chassis_boom_link
- removed link stick_bucket_link
- added link Link_EE, mass 1; visual sphere radius=0.0001
- added link base, mass 1
- added link kanan, mass 1072.99833902132; collision mesh filename=meshes/kanan.STL; visual mesh filename=meshes/kanan.STL
- added link kiri, mass 1072.99833917086; collision mesh filename=meshes/kiri.STL; visual mesh filename=meshes/kiri.STL
- added link link2, mass 14373.8102967852; collision mesh filename=meshes/link2.STL; visual mesh filename=meshes/link2.STL
- added link link3, mass 2653.35957715292; collision mesh filename=meshes/link3.STL; visual mesh filename=meshes/link3.STL
- added link link4, mass 112.346086234288; collision mesh filename=meshes/link4.STL; visual mesh filename=meshes/link4.STL
- added link link5, mass 641.54889296027; collision mesh filename=meshes/link5.STL; visual mesh filename=meshes/link5.STL
- link base_link: mass 139411.733176679 -> 1992.01573661862
Joints:
- removed joint base_chassis_joint
- removed joint boom_stick_joint
- removed joint chassis_boom_joint
- removed joint stick_bucket_joint
- added joint Joint_EE: type fixed, parent link5, child Link_EE, origin xyz=2 0 -0.75 rpy=0 0 0, axis 1 0 0
- added joint base_to_base: type fixed, parent base, child base_link, origin xyz=0 0 0 rpy=0 0 0, axis 0 0 1
- added joint base_to_kanan: type continuous, parent base_link, child kanan, origin xyz=0 0 0 rpy=0 0 0, axis 0 1 0
- added joint base_to_kiri: type continuous, parent base_link, child kiri, origin xyz=0 0 0 rpy=0 0 0, axis 0 1 0
- added joint link2_to_base: type revolute, parent base_link, child link2, origin xyz=-0.8585 -0.0825 1.466 rpy=0 0 0.075368, axis 0 0 1, limit lower=-3.1 upper=3.1 effort=300 velocity=0.1
- added joint link3_to_link2: type revolute, parent link2, child link3, origin xyz=1.306 -0.015884 -0.544 rpy=0 0.34319 -0.075368, axis 0 1 0, limit lower=-0.954 upper=1.03 effort=300 velocity=0.1
- added joint link4_to_link3: type revolute, parent link3, child link4, origin xyz=6.9891 0 2.5506 rpy=0 0.40612 0, axis 0 1 0, limit lower=-0.1214 upper=1.51 effort=300 velocity=0.1
- added joint link5_to_link4: type revolute, parent link4, child link5, origin xyz=2.6047 0 0.78507 rpy=0 -0.88131 0, axis 0 1 0, limit lower=-0.32 upper=3.14 effort=300 velocity=0.1
